File: Hardware/KiCAD/UI/UI-Bridge.sch (KiCad schematic (older format))
At the start: 14 parts

Commit message: Monitor is now better
A little memory leaks.
Updated hardware from piotr.
Parts:
- X?: value CRYSTAL -> 11.0592MHz
Other:
- note added: "DODAĆ LCD z PWM, PRZYCISKI, ENCODER Z PRZYCISKIEM, POWER(?), PILOT(?)\nWYPROWADZENIA "FUTURE""
- note removed: "DODAĆ LCD z PWM, PRZYCISKI, ENCODER Z PRZYCISKIEM, POWER(?), PILOT(?)"
Changed lines of the file:
@@
 LIBS:contrib
 LIBS:valves
+LIBS:UI-Bridge-cache
 EELAYER 27 0
 EELAYER END
@@
 Sheet 1 1
 Title ""
-Date "30 aug 2015"
+Date "16 apr 2016"
 Rev ""
 Comp ""
@@
 P 3550 3850
 F 0 "X?" H 3550 3975 50  0000 C CNN
-F 1 "CRYSTAL" H 3550 3725 40  0000 C CNN
+F 1 "11.0592MHz" H 3550 3725 40  0000 C CNN
 F 2 "" H 3550 3850 60  0000 C CNN
 F 3 "" H 3550 3850 60  0000 C CNN
@@
 RESET
 Text Notes 6100 2300 0    60   ~ 0
-DODAĆ LCD z PWM, PRZYCISKI, ENCODER Z PRZYCISKIEM, POWER(?), PILOT(?)
+DODAĆ LCD z PWM, PRZYCISKI, ENCODER Z PRZYCISKIEM, POWER(?), PILOT(?)\nWYPROWADZENIA "FUTURE"
 $EndSCHEMATC
